File: Hardware/Revolute.kicad_pcb (KiCad board)
At the start: 4 copper layers, 17.3 x 11.4 mm, 31 parts, among them J1 USB_A, U1 nRF52840_aQFN73, U2 debug_ports, U3 AP2112K-3.3, X1 32MHZ, X2 32.768 kHz

Commit message: version 2 base pcb
Parts:
- removed U2: debug_ports, Library:Debug pin cluster
- added U4: debug_ports, Library:Debug pin cluster, F.Cu at (173.1, 81.9)
Connections:
- U1 pad G1: unconnected-(U1-PadG1) -> P0.26
- U1 pad H2: unconnected-(U1-PadH2) -> P0.27
Routing:
- net P0.26: track 0.00 -> 14.5 mm, vias 0 -> 2
- net P0.27: track 0.00 -> 12.1 mm, vias 0 -> 2
- net P1.02: track 9.16 -> 0.00 mm, vias 2 -> 0
- net P1.01: track 5.84 -> 0.00 mm, vias 2 -> 0
- net VDD_nRF: track 21.5 -> 25.1 mm
- net swc: track 7.03 -> 3.69 mm
- net swd: track 5.06 -> 1.95 mm
- net GND: track 26.1 -> 24.5 mm, vias 19 -> 17
- net Net-(U1-P0.18/~{RESET}): track 11.4 -> 10.0 mm, vias 2 -> 1
- net VBUS: track 35.4 -> 34.0 mm
- net Net-(J1-D-): track 14.3 -> 13.5 mm
