File: Hardware/MainPCB/Revolute.kicad_pcb (KiCad board)
At the start: 4 copper layers, 17.3 x 11.4 mm, 31 parts, among them J1 USB_A, U1 nRF52840_aQFN73, U3 AP2112K-3.3, U4 debug_ports, X1 32MHZ, X2 32.768 kHz

Commit message: updated pcb design
Parts:
- removed C3: 0.8pF, Capacitor_SMD:C_0402_1005Metric
- added ?: , , F.Cu at (180.8, 84.6)
- added ?: , , F.Cu at (181.3, 83.4)
- moved ? 9.15 mm to (181.2, 91.9), turned to 180 degrees
- moved ? 6.75 mm to (181.2, 90.7), turned to 180 degrees
- moved C13 3.45 mm to (178.0, 87.5), turned to -90 degrees
- moved C11 1.09 mm to (177.1, 87.5), turned to 90 degrees
- moved C16 1.04 mm to (181.2, 85.8), turned to 180 degrees
- moved U3 0.85 mm to (180.3, 88.1)
- moved R1 0.81 mm to (177.4, 90.1)
- moved U4 0.52 mm to (172.5, 81.9)
- moved C9 0.28 mm to (177.5, 89.0)
- moved D1 0.25 mm to (179.8, 91.2)
- moved C1 0.12 mm to (177.9, 86.0)
Connections:
- U1 pad P23: unconnected-(U1-P1.07-PadP23) -> P1.07
- U1 pad T23: unconnected-(U1-P1.05-PadT23) -> P1.05
Routing:
- net P1.05: track 0.00 -> 10.6 mm, vias 0 -> 2
- net P1.07: track 0.00 -> 10.2 mm, vias 0 -> 2
- net GND: track 24.5 -> 19.9 mm, vias 17 -> 15
- net VDD_nRF: track 19.9 -> 18.0 mm, vias 7 -> 6
- net Net-(U1-ANT): track 1.80 -> 0.00 mm
- net VBUS: track 34.2 -> 32.9 mm
- net swd: track 1.95 -> 1.03 mm
- net BLUE_LED: track 9.62 -> 8.86 mm
- net Net-(U1-DEC4): track 11.0 -> 10.4 mm
- net P0.27: track 12.1 -> 12.7 mm
- net Net-(D1-K): track 1.30 -> 1.88 mm
Other:
- board size 17.3 x 11.4 mm -> 16.8 x 11.4 mm

Commit message: made pcb smaller
Parts:
- moved U4 0.35 mm to (172.5, 81.6)
Routing:
- net VBUS: track 32.9 -> 30.0 mm
- net GND: track 19.9 -> 17.6 mm, vias 15 -> 12
- net VDD_nRF: track 18.0 -> 17.1 mm, vias 6 -> 5
- net Net-(J1-D-): track 13.6 -> 12.8 mm
Other:
- board size 16.8 x 11.4 mm -> 16.8 x 10.7 mm
