File: Hardware/Wireless/Revolutetestboard.kicad_pcb (KiCad board)
At the start: 4 copper layers, 54 x 85.6 mm, 261 parts, among them J1 Conn_01x02_Pin, J2 Conn_01x02_Pin, J3 Conn_01x02_Pin, J4 Conn_01x04_Socket, J5 Conn_01x02_Pin, J6 Conn_01x04_Pin, J7 USB_C_Receptacle_USB2.0, J8 USB_C_Receptacle_USB2.0, Q1 NMOS-CSD17381F4, Q10 PMOS-BSS84, Q2 NMOS-CSD17381F4, Q3 PMOS-CSD25483F4, Q4 PMOS-CSD25483F4, Q5 PMOS-CSD25483F4, Q7 PMOS-BSS84, Q8 IRLML6344, Q9 PMOS-BSS84, SW1 SW_DIP_x06, SW2 SW_DPDT_x2, SW3 SW_DIP_x06, SW4 SW_Push, SW5 SW_DPDT_x2, SW6 SW_DPDT_x2, U1 BQ27427, U10 battery_charger, U11 nRF52840_aQFN73, U12 TS5A3159AYZPR, U13 BQ27427, U14 TPS22910A, U15 A3144e, U16 A3144e, U18 pogopins, U19 LSM6DS3, U2 nrf52833_qfn40, U20 TPS54202DDC, U21 TPS54202DDC, U22 STM32F103CBTx, U23 AP2112K-3.3, U24 Conn_01x14_Socket, U3 Conn_01x14_Socket, U4 TPS709, U5 AS5600, U6 BQ25180, U7 LSM6DSO, U8 TS5A3159AYZPR, U9 TPS22910A, X1 32.768 kHz, X2 32MHZ, X3 32.768 kHz, X4 32MHZ, Y1 32.768KHZ, Y2 8Mhz

Commit message: routing session 1
Parts:
- TP10, TP3: moved to B.Cu
- moved TP2 56.3 mm to (157.8, 117.0)
- moved TP3 55.9 mm to (156.8, 126.0), turned to 180 degrees
- moved R32 9.07 mm to (114.7, 121.2), turned to 0 degrees
- moved JP4 7.93 mm to (110.9, 113.4), turned to 180 degrees
- moved U12 6.85 mm to (114.4, 119.5), turned to 0 degrees
- moved C54 6.81 mm to (115.5, 119.9), turned to -90 degrees
- moved R14 5.80 mm to (155.5, 136.7), turned to 90 degrees
- moved TP10 5.61 mm to (115.0, 122.8), turned to 180 degrees
- moved C78 5.44 mm to (144.7, 132.7), turned to -45 degrees
- moved C25 5.14 mm to (153.8, 134.6), turned to 0 degrees
- moved C70 4.81 mm to (135.3, 131.8), turned to -135 degrees
- moved TP7 4.80 mm to (118.2, 112.6)
- moved R36 4.53 mm to (122.8, 109.5)
- moved C19 3.80 mm to (148.2, 136.1)
- moved C22 3.80 mm to (150.9, 134.5)
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Routing:
- net /dbg/USBDM2: track 0.00 -> 23.2 mm, vias 0 -> 3
- net /dbg/USBDP2: track 0.00 -> 22.7 mm, vias 0 -> 1
- net 5V: track 0.00 -> 16.0 mm, vias 0 -> 4
- net GND: track 0.00 -> 15.7 mm, vias 0 -> 10
- net 5V(2): track 0.00 -> 14.7 mm, vias 0 -> 4
- net /pod/3V: track 0.00 -> 13.3 mm, vias 0 -> 9
- net Net-(Q9-D): track 0.00 -> 11.9 mm
- net /dbg/USBDP: track 0.00 -> 10.9 mm, vias 0 -> 2
- net /dbg/USBDM: track 0.00 -> 10.7 mm, vias 0 -> 1
- net /rev/VDD_nRF: track 0.00 -> 10.4 mm, vias 0 -> 6
- net Net-(JP6-A): track 0.00 -> 10.3 mm
- net /rev/P0.17: track 0.00 -> 8.40 mm
- net /rev/VBUS: track 0.00 -> 7.91 mm, vias 0 -> 3
- net Net-(U22-PC15): track 0.00 -> 7.62 mm
- net /rev/MOS_VDD: track 0.00 -> 7.53 mm, vias 0 -> 6
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- added copper zone on F.Cu, net /pod/3V
- added copper zone on F.Cu, net /pod/44E
- added copper zone on F.Cu, net /pod/5V
- added copper zone on F.Cu, net /pod/BAT_P
- added copper zone on F.Cu, net /pod/COM
- added copper zone on F.Cu, net /pod/SAFE_5V
- added copper zone on F.Cu, net /pod/V
- added copper zone on F.Cu, net /pod/VBUS
- added copper zone on F.Cu, net /rev/+
- added copper zone on F.Cu, net /rev/-
- added copper zone on F.Cu, net /rev/COM
- added copper zone on F.Cu, net /rev/MOS_VDD
- added copper zone on F.Cu, net /rev/VDD_nRF
- added copper zone on F.Cu, net /rev/vSYSTEM
- added copper zone on F.Cu, net 3.3V
- added copper zone on F.Cu, net Net-(C35-Pad2)
- added copper zone on F.Cu, net Net-(JP2-A)
- added copper zone on F.Cu, net Net-(JP4-B)
- added copper zone on F.Cu, net Net-(JP5-B)
- added copper zone on F.Cu, net Net-(U20-FB)
- added copper zone on F.Cu, net Net-(U21-FB)
- added copper zone on F.Cu, net Net-(U21-SW)

Commit message: route2
Parts:
- added U25: TLV493D, Library:SOT-23-6-Small, F.Cu at (143.5, 128.0)
- moved R12 6.99 mm to (148.9, 126.0), turned to 180 degrees
- moved R11 6.91 mm to (147.3, 125.6), turned to -90 degrees
- moved U5 1.99 mm to (148.8, 130.3), turned to 90 degrees
- moved C22 1.59 mm to (151.6, 135.9), turned to -90 degrees
- moved C18 1.30 mm to (144.6, 124.9), turned to 90 degrees
- moved R4 0.75 mm to (149.1, 120.5)
- moved X1 0.59 mm to (151.7, 125.3)
- moved C2 0.58 mm to (150.2, 125.8)
- moved C3 0.58 mm to (152.1, 126.5)
- moved C19 0.56 mm to (147.7, 135.9)
- moved U4 0.56 mm to (149.7, 135.9)
- moved R6 0.11 mm to (154.0, 125.7)
- moved C4 0.09 mm to (149.8, 124.3)
- moved C20 0.07 mm to (145.5, 125.0), turned to 90 degrees
Routing:
- net /dbg/swd: track 2.21 -> 9.72 mm
- net /pod/VBUS: track 4.46 -> 6.38 mm, vias 1 -> 4
- net /rev/P0.09: track 4.00 -> 5.86 mm, vias 0 -> 2
- net Net-(U7-CS): track 0.00 -> 1.78 mm
- net /pod/MOS_VDD: track 5.18 -> 6.91 mm, vias 0 -> 2
- net Net-(U2-DEC1): track 0.00 -> 1.67 mm
- net /pod/V: track 7.28 -> 8.95 mm, vias 0 -> 2
- net /rev/P0.10: track 4.00 -> 5.62 mm, vias 0 -> 2
- net 5V(2): track 14.7 -> 16.0 mm, vias 4 -> 5
- net /dbg/swc: track 3.27 -> 4.51 mm, vias 3 -> 4
- net /rev/MOS_VDD: track 7.53 -> 6.30 mm, vias 6 -> 5
- net Net-(U1-BIN): track 0.00 -> 1.23 mm
- net /pod/D-: track 0.00 -> 1.18 mm, vias 0 -> 1
- net /pod/swd: track 0.46 -> 1.62 mm, vias 1 -> 2
- net /dbg/USBDP2: track 22.7 -> 23.8 mm, vias 1 -> 2
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
Commit message: new route
Parts:
- TP1: moved to B.Cu
- moved TP1 54.2 mm to (150.7, 130.5), turned to 180 degrees
- moved D32 50.3 mm to (140.5, 71.5), turned to -90 degrees
- moved D31 47.3 mm to (138.4, 71.5), turned to -90 degrees
- moved D26 45.2 mm to (127.9, 71.4), turned to -90 degrees
- moved D30 44.3 mm to (136.3, 71.5), turned to -90 degrees
- moved D25 42.2 mm to (125.8, 71.4), turned to -90 degrees
- moved D29 41.3 mm to (134.2, 71.5), turned to -90 degrees
- moved R46 40.8 mm to (119.6, 129.9), turned to -90 degrees
- moved D24 39.3 mm to (123.7, 71.4), turned to -90 degrees
- moved D19 38.7 mm to (113.6, 72.2), turned to -62 degrees
- moved D28 38.3 mm to (132.0, 71.5), turned to -90 degrees
- moved D23 36.3 mm to (121.5, 71.4), turned to -90 degrees
- moved D27 35.3 mm to (129.9, 71.5), turned to -90 degrees
- moved D18 34.9 mm to (112.0, 73.5), turned to -42 degrees
- moved D22 33.4 mm to (119.4, 71.4), turned to -90 degrees
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Routing:
- net Net-(BT2-+): track 0.00 -> 22.9 mm
- net /pod/ARGBLED_5V: track 0.00 -> 18.6 mm, vias 0 -> 27
- net Net-(SW2A-B): track 0.66 -> 18.3 mm
- net /pod/BAT_P: track 0.73 -> 6.38 mm, vias 2 -> 3
- net Net-(J5-Pin_1): track 0.00 -> 5.07 mm
- net Net-(BT1-+): track 0.00 -> 3.95 mm
- net /dbg/USBDP2: track 23.8 -> 27.2 mm, vias 2 -> 3
- net /pod/VBUS: track 6.38 -> 9.37 mm, vias 4 -> 7
- net Net-(D6-DI): track 0.00 -> 2.75 mm, vias 0 -> 2
- net Net-(J1-Pin_1): track 0.00 -> 2.64 mm, vias 0 -> 1
- net Net-(D8-DO): track 0.00 -> 1.71 mm
- net Net-(D7-DO): track 0.00 -> 1.71 mm
- net Net-(D6-DO): track 0.00 -> 1.71 mm
- net Net-(D12-DO): track 0.00 -> 1.71 mm
- net Net-(D11-DO): track 0.00 -> 1.71 mm
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