File: Hardware/Wireless/Revolutetestboard.kicad_pcb (KiCad board)
At the start: 4 copper layers, 54 x 85.6 mm, 262 parts, among them J1 Conn_01x02_Pin, J2 Conn_01x02_Pin, J3 Conn_01x02_Pin, J4 Conn_01x04_Socket, J5 Conn_01x02_Pin, J6 Conn_01x04_Pin, J7 USB_C_Receptacle_USB2.0, J8 USB_C_Receptacle_USB2.0, Q1 NMOS-CSD17381F4, Q10 PMOS-BSS84, Q2 NMOS-CSD17381F4, Q3 PMOS-CSD25483F4, Q4 PMOS-CSD25483F4, Q5 PMOS-CSD25483F4, Q7 PMOS-BSS84, Q8 IRLML6344, Q9 PMOS-BSS84, SW1 SW_DIP_x06, SW2 SW_DPDT_x2, SW3 SW_DIP_x06, SW4 SW_Push, SW5 SW_DPDT_x2, SW6 SW_DPDT_x2, U1 BQ27427, U10 battery_charger, U11 nRF52840_aQFN73, U12 TS5A3159AYZPR, U13 BQ27427, U14 TPS22910A, U15 A3144e, U16 A3144e, U18 pogopins, U19 LSM6DS3, U2 nrf52833_qfn40, U20 TPS54202DDC, U21 TPS54202DDC, U22 STM32F103CBTx, U23 AP2112K-3.3, U24 Conn_01x14_Socket, U25 TLV493D, U3 Conn_01x14_Socket, U4 TPS709, U5 AS5600, U6 BQ25180, U7 LSM6DSO, U8 TS5A3159AYZPR, U9 TPS22910A, X1 32.768 kHz, X2 32MHZ, X3 32.768 kHz, X4 32MHZ, Y1 32.768KHZ, Y2 8Mhz

Commit message: route
Parts:
- moved TP7 0.20 mm to (118.4, 112.7)
Routing:
- net Net-(BT2-+): track 22.9 -> 0.00 mm
- net Net-(SW2A-B): track 18.3 -> 0.66 mm
- net /pod/BAT_P: track 6.38 -> 0.73 mm, vias 3 -> 2
- net Net-(J5-Pin_1): track 5.07 -> 0.00 mm
- net /pod/VBUS: track 9.37 -> 6.38 mm, vias 7 -> 4
- net /dbg/USBDP2: track 27.2 -> 24.4 mm, vias 3 -> 2
- net Net-(J1-Pin_1): track 2.64 -> 0.00 mm, vias 1 -> 0
- net /rev/vBAT: track 1.53 -> 3.08 mm, vias 0 -> 2
- net /rev/VBUS: track 7.91 -> 9.40 mm, vias 4 -> 3
- net /pod/P0.14: track 0.00 -> 1.31 mm, vias 0 -> 2
- net /pod/IN_TS5A3159AYZPR: track 0.00 -> 1.28 mm, vias 0 -> 2
- net /pod/3V: track 13.0 -> 11.8 mm, vias 13 -> 9
- net /pod/5V: track 0.00 -> 1.00 mm, vias 0 -> 2
- net /pod/MOS_EN: track 2.14 -> 3.14 mm, vias 1 -> 2
- net /rev/COM: track 0.00 -> 0.93 mm, vias 0 -> 1
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
Commit message: added some zones
Routing:
- net /rev/P0.17: track 9.43 -> 12.0 mm, vias 1 -> 4
- net /rev/P0.15: track 8.14 -> 10.2 mm, vias 2 -> 4
- net /rev/VBUS: track 9.40 -> 10.2 mm, vias 3 -> 4
- net /rev/VDD_nRF: track 10.4 -> 11.0 mm, vias 6 -> 7
- net Net-(U2-DEC4): track 3.26 -> 3.69 mm, vias 0 -> 1
- added copper zone on In2.Cu, net /pod/3V
- added copper zone on In2.Cu, net /rev/MOS_VDD
- added copper zone on In2.Cu, net /rev/VDD_nRF
- added copper zone on In2.Cu, net /rev/vSYSTEM
- added copper zone on In2.Cu, net 3.3V
- added copper zone on In2.Cu, net 5V
- added copper zone on In2.Cu, net 5V(2)

Commit message: route
Connections:
- J4 pad 4: unconnected-(J4-Pin_4-Pad4) -> /rev/P0.17
Routing:
- net /pod/BATM: track 1.61 -> 25.6 mm
- net led: track 4.49 -> 22.1 mm
- net /pod/swd: track 1.64 -> 17.1 mm
- net /pod/5V: track 1.00 -> 15.8 mm
- net /dbg/swd: track 9.72 -> 24.5 mm
- net /pod/VBUS: track 6.38 -> 19.1 mm
- net /pod/swc: track 1.64 -> 14.3 mm
- net /dbg/swc: track 4.51 -> 17.0 mm
- net /pod/V: track 8.95 -> 20.5 mm
- net /pod/BAT_P: track 0.73 -> 9.18 mm
- net /rev/swd: track 2.52 -> 9.95 mm
- net /rev/RESET: track 0.80 -> 6.43 mm, vias 1 -> 2
- net /rev/swc: track 2.57 -> 7.99 mm
- net /dbg/USBDP2: track 24.4 -> 25.8 mm, vias 2 -> 3
- net Net-(J4-Pin_2): track 0.00 -> 1.22 mm, vias 0 -> 1
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
Commit message: routed
Parts:
- added J9: Conn_01x04_Socket, Connector_PinSocket_2.54mm:PinSocket_1x04_P2.54mm_Vertical, F.Cu at (121.9, 139.2)
- moved R4 0.27 mm to (149.1, 120.7)
Routing:
- net /pod/COM: track 1.99 -> 67.2 mm, vias 1 -> 4
- net /pod/SCL: track 2.85 -> 62.1 mm
- net /pod/SDA: track 3.23 -> 59.9 mm
- net /rev/P0.15: track 10.2 -> 55.1 mm, vias 4 -> 6
- net /pod/vBATM: track 0.79 -> 43.9 mm
- net /rev/FLEX_LED: track 2.68 -> 43.4 mm, vias 3 -> 5
- net /rev/swd: track 9.95 -> 48.3 mm, vias 3 -> 6
- net /pod/VBUS: track 19.1 -> 57.0 mm, vias 4 -> 5
- net /rev/D+: track 1.89 -> 39.3 mm, vias 2 -> 5
- net /rev/P0.17: track 12.0 -> 48.6 mm
- net /pod/ARGBLED_5V: track 19.3 -> 55.5 mm
- net /rev/VBUS: track 10.2 -> 44.4 mm, vias 4 -> 8
- net Net-(D6-DI): track 2.75 -> 35.7 mm
- net /dbg/swc: track 17.0 -> 48.0 mm
- net /rev/D-: track 1.96 -> 31.2 mm, vias 2 -> 5
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- added copper zone on In2.Cu, net /pod/ARGBLED_5V
- added copper zone on F.Cu, net Net-(C36-Pad2)
