File: Hardware/Wireless/Revolutetestboard.kicad_sch (KiCad schematic)
At the start: 102 parts, among them J1 -, J2 +, J3 USB_C_Receptacle_USB2.0, J4 Conn_01x02_Pin, J5 USB_C_Receptacle_USB2.0, Q1 NMOS, Q2 NMOS-CSD17381F4, Q3 NMOS-CSD17381F4, Q4 PMOS-CSD25483F4, Q5 PMOS-CSD25483F4, SW1 SW_DIP_x05, U11 LSM6DSO, U12 STM32F103C8Tx, U13 AP2112K-3.3, U14 Conn_01x14_Socket, U2 Button, U2 nrf52833_qfn40, U3 AS5600, U4 MIC5504, U5 BQ24075RGT, U7 Conn_01x14_Socket, X1 32.768 kHz, X2 32MHZ, Y1 32.768KHZ, Y2 8Mhz

Commit message: new flex and new pcbs
Parts:
- removed Q1: NMOS, Library:Mosfet0402, symbol Simulation_SPICE:NMOS
- added J6: Conn_01x04_Socket, Connector_PinSocket_2.54mm:PinSocket_1x04_P2.54mm_Vertical, symbol Connector:Conn_01x04_Socket
- added JP6: Jumper_3_Bridged12, Jumper:SolderJumper-3_P1.3mm_Bridged12_RoundedPad1.0x1.5mm, symbol Jumper:Jumper_3_Bridged12
- added Q1: PMOS-CSD25483F4, Library:Mosfet0402, symbol Simulation_SPICE:PMOS
- added R23: 2M, Library:Resistor_0402_1005M-nosilk, symbol Device:R
- added SW2: SW_Push, Library:16mmCompButton, symbol Switch:SW_Push
- added TP1, TP10, TP11, TP12, TP13, TP2, TP3, TP4, TP5, TP6, TP7, TP8, TP9: TestPoint, TestPoint:TestPoint_Pad_D1.0mm, symbol Connector:TestPoint
Connections:
- net 3.3V: now also TP5.1
- net 5V: now also TP3.1
- net A5: now also TP6.1
- net B14: now also TP7.1
- net D+: now also SW1.4
- net D-: now also SW1.5
- net GND: now also J6.1 (Pin_1), R23.2, SW2.2, TP2.1, TP4.1
- net MOS_EN: now also Q1.1 (G), R23.1
- net MOS_VDD: now also JP6.3 (B), Q1.3 (D), TP11.1, TP9.1
- net OUT: now also TP8.1
- net P0.15: now also J6.3 (Pin_3)
- net P0.17: now also J6.4 (Pin_4)
- net P0.28: now also SW2.1
- net RESET: now also TP1.1
- net VBUS: now also SW1.1, TP12.1
- net VDD_nRF: now also JP6.1 (A), Q1.2 (S), TP10.1
- net swc: now also SW1.2
- net swd: now also SW1.3
- net vBAT: now also TP13.1
- new net: J6.2 (Pin_2), JP6.2 (C)

Commit message: unrouted test board
Parts:
- removed BT1: Battery_Cell, Battery:BatteryHolder_Keystone_1060_1x2032, symbol Device:Battery_Cell
- removed C1, C6, C8: 4.7uF, Library:Capacitor_0402_1005M-nosilk, symbol Device:C_Small
- removed C10, C4: 12pF, Capacitor_SMD:C_0402_1005Metric, symbol Device:C
- removed C11: 47nF, Library:Capacitor_0402_1005M-nosilk, symbol Device:C_Small
- removed C12: 2.2uF, Library:Capacitor_0402_1005M-nosilk, symbol Device:C_Small
- removed C13, C5: 100nF, Library:Capacitor_0402_1005M-nosilk, symbol Device:C_Small
- removed C14: 820pF, Library:Capacitor_0402_1005M-nosilk, symbol Device:C_Small
- removed C15: 1pF, Library:Capacitor_0402_1005M-nosilk, symbol Device:C_Small
- removed C16, C17, C2, C3: 12pF, Library:Capacitor_0402_1005M-nosilk, symbol Device:C_Small
- removed C18: 100pF, Library:Capacitor_0402_1005M-nosilk, symbol Device:C_Small
- removed C19: 1.2pF, Library:Capacitor_0402_1005M-nosilk, symbol Device:C_Small
- removed C20: 100nF, Library:Capacitor_0402_1005M-nosilk, symbol Device:C
- removed C21: 1uF, Library:Capacitor_0402_1005M-nosilk, symbol Device:C
- removed C22, C23, C24, C7, C9: 1uF, Library:Capacitor_0402_1005M-nosilk, symbol Device:C_Small
- removed C25, C26: 10uF, Capacitor_SMD:C_0402_1005Metric, symbol Device:C_Small
- removed C27, C28, C30, C31, C33: 100nF, Capacitor_SMD:C_0402_1005Metric, symbol Device:C
- removed C29, C32: 10uF, Capacitor_SMD:C_0402_1005Metric, symbol Device:C
- removed C34, C35: 22pf, Capacitor_SMD:C_0402_1005Metric, symbol Device:C
- removed D1: BLUE, LED_SMD:LED_0402_1005Metric, symbol Device:LED_Small
- removed D2: LED, LED_SMD:LED_0402_1005Metric, symbol Device:LED
- removed D3: BLUE, LED_SMD:LED_0402_1005Metric, symbol Device:LED
- removed D4: White, LED_SMD:LED_0402_1005Metric, symbol Device:LED
- removed J1: -, Library:Pogo-pin-recepticle, symbol Connector:Conn_01x01_Socket
- removed J2: +, Library:Pogo-pin-recepticle, symbol Connector:Conn_01x01_Socket
- removed J3, J5: USB_C_Receptacle_USB2.0, Library:USB-C_C168688, symbol Library:USB_C_Receptacle_USB2.0
- removed J4: Conn_01x02_Pin, Connector_PinSocket_2.54mm:PinSocket_1x02_P2.54mm_Vertical, symbol Connector:Conn_01x02_Pin
- removed J6: Conn_01x04_Socket, Connector_PinSocket_2.54mm:PinSocket_1x04_P2.54mm_Vertical, symbol Connector:Conn_01x04_Socket
- removed JP1: SolderJumper_2_Open, Jumper:SolderJumper-2_P1.3mm_Open_RoundedPad1.0x1.5mm, symbol Jumper:SolderJumper_2_Open
- removed JP2, JP3: Jumper_3_Open, Jumper:SolderJumper-3_P1.3mm_Open_RoundedPad1.0x1.5mm, symbol Jumper:Jumper_3_Open
- removed JP4: Jumper_2_Open, Jumper:SolderJumper-2_P1.3mm_Open_RoundedPad1.0x1.5mm, symbol Jumper:Jumper_2_Open
- removed JP5: Jumper_2_Bridged, Jumper:SolderJumper-2_P1.3mm_Bridged_RoundedPad1.0x1.5mm, symbol Jumper:Jumper_2_Bridged
- removed JP6: Jumper_3_Bridged12, Jumper:SolderJumper-3_P1.3mm_Bridged12_RoundedPad1.0x1.5mm, symbol Jumper:Jumper_3_Bridged12
- removed L1: 10uH, Inductor_SMD:L_0402_1005Metric, symbol Device:L
- removed L2: 15nH, Inductor_SMD:L_0402_1005Metric, symbol Device:L
- removed L3: 4.7nH, Inductor_SMD:L_0402_1005Metric, symbol Device:L
- removed L4: 2.2nH, Inductor_SMD:L_0402_1005Metric, symbol Device:L
- removed Q1, Q4, Q5: PMOS-CSD25483F4, Library:Mosfet0402, symbol Simulation_SPICE:PMOS
- removed Q2, Q3: NMOS-CSD17381F4, Library:Mosfet0402, symbol Simulation_SPICE:NMOS
- removed R10, R7: 0Ω, Library:Resistor_0402_1005M-nosilk, symbol Device:R_Small
- removed R11: 10k, Library:Resistor_0402_1005M-nosilk, symbol Device:R_Small
- removed R12, R13, R21, R22: 5.1K, Resistor_SMD:R_0402_1005Metric, symbol Device:R
- removed R14, R15, R16: 10k, Resistor_SMD:R_0402_1005Metric, symbol Device:R
- removed R17: 1.5K, Resistor_SMD:R_0402_1005Metric, symbol Device:R
- removed R18, R19: 510Ω, Resistor_SMD:R_0402_1005Metric, symbol Device:R
- removed R20: 1M, Resistor_SMD:R_0402_1005Metric, symbol Device:R
- removed R23: 2M, Library:Resistor_0402_1005M-nosilk, symbol Device:R
- removed R3: 100K, Library:Resistor_0402_1005M-nosilk, symbol Device:R_Small
- removed R4: 1.1k, Library:Resistor_0402_1005M-nosilk, symbol Device:R_Small
- removed R5: 590, Library:Resistor_0402_1005M-nosilk, symbol Device:R_Small
- removed R6, R8: 4.7K, Library:Resistor_0402_1005M-nosilk, symbol Device:R
- removed R9: 1.5k, Library:Resistor_0402_1005M-nosilk, symbol Device:R_Small
- removed S1: Button 3*3*1.5, Library:button 3x3, symbol Switch:SW_Push
- removed SW1: SW_DIP_x05, Button_Switch_SMD:SW_DIP_SPSTx05_Slide_KingTek_DSHP05TS_W7.62mm_P1.27mm, symbol Switch:SW_DIP_x05
- removed SW2: SW_Push, Library:16mmCompButton, symbol Switch:SW_Push
- removed TH1: 10K, Library:Resistor_0402_1005M-nosilk, symbol Device:Thermistor
- removed TP1, TP10, TP11, TP12, TP13, TP3, TP4, TP5, TP6, TP7, TP8, TP9: TestPoint, TestPoint:TestPoint_Pad_D1.0mm, symbol Connector:TestPoint
- removed U1: ~, Package_BGA:Texas_DSBGA-9_1.62mmx1.58mm_Layout3x3_P0.5mm, symbol Library:BQ27427
- removed U11: LSM6DSO, Package_LGA:LGA-14_3x2.5mm_P0.5mm_LayoutBorder3x4y, symbol Sensor_Motion:LSM6DS3
- removed U12: STM32F103C8Tx, Package_QFP:LQFP-48_7x7mm_P0.5mm, symbol MCU_ST_STM32F1:STM32F103C8Tx
- removed U13: AP2112K-3.3, Package_TO_SOT_SMD:SOT-23-5, symbol Regulator_Linear:AP2112K-3.3
- removed U14, U7: Conn_01x14_Socket, Library:FPC, symbol Connector:Conn_01x14_Socket
- removed U2 (x4): Button, Library:SMDButton, symbol Library:Button
- removed U2: nrf52833_qfn40, Library:QFN-40-1EP_5x5mm_P0.4mm_EP3.6x3.6mm, symbol Library:nrf52833_qfn40
- removed U3: AS5600, Library:SOIC-8-1EP_3.9x4.9mm_P1.27mm_EP2.514x3.2mm, symbol Library:AS5600
- removed U4: MIC5504, Library:TDFN-4, symbol ESP32-eagle-import:MIC5504
- removed U5: BQ24075RGT, Package_DFN_QFN:VQFN-16-1EP_3x3mm_P0.5mm_EP1.6x1.6mm, symbol Battery_Management:BQ24075RGT
- removed X1: 32.768 kHz, Library:Crystal_SMD_2012-2Pin_2.0x1.2mm, symbol Device:Crystal_Small
- removed X2: 32MHZ, Library:Crystal_SMD_2016-4Pin_2.0x1.6mm, symbol Device:Crystal_GND24_Small
- removed Y1: 32.768KHZ, Crystal:Crystal_SMD_3215-2Pin_3.2x1.5mm, symbol Device:Crystal
- removed Y2: 8Mhz, Crystal:Crystal_SMD_3225-4Pin_3.2x2.5mm, symbol Device:Crystal_GND24_Small
- added J1: Conn_01x02_Pin, Connector_PinHeader_2.54mm:PinHeader_1x02_P2.54mm_Vertical, symbol Connector:Conn_01x02_Pin
- added SW1, SW3: SW_DIP_x06, Button_Switch_SMD:SW_DIP_SPSTx06_Slide_Copal_CHS-06B_W7.62mm_P1.27mm, symbol Switch:SW_DIP_x06
- added SW2: SW_DPDT_x2, Library:MST-12C05 SLIDEBUTTON, symbol Switch:SW_DPDT_x2
- R1: value 10k -> 0r; footprint Library:Resistor_0402_1005M-nosilk -> Library:0402
- R2: value 1.5k -> 0r; footprint Library:Resistor_0402_1005M-nosilk -> Library:0402; ID 138 -> 110
- renumbered TP2 to TP1
Connections:
- net GND: now also R1.2; no longer R1.1, R2.1
- net at R2.2: now also SW2.2 (B)
- new net: J1.1 (Pin_1), SW2.3 (C)
- new net dbg/5v: SW1.12, SW3.12
- new net dbg/led: SW1.7, SW3.7
- new net dbg/pass D+: SW1.9, SW3.9
- new net dbg/pass D-: SW1.8, SW3.8
- new net dbg/swc: SW1.11, SW3.11
- new net dbg/swd: SW1.10, SW3.10
- new net pod/com: J1.2 (Pin_2), SW2.1 (A)
- new net pod/d+: SW3.4
- new net pod/d-: SW3.5
- new net pod/swc: SW3.2
- new net pod/swd: SW3.3
- new net pod/vbus: SW3.1
- new net rev/5V: SW1.1
- new net rev/D-: SW1.5
- new net rev/d+: SW1.4
- new net rev/led: SW1.6
- new net rev/pogo 1: R2.1
- new net rev/pogo 2: R1.1
- new net rev/swc: SW1.2
- new net rev/swd: SW1.3
- no-connect marks 10 -> 0
Other:
- added sheet dbg (dbg.kicad_sch)
- added sheet pod (pod.kicad_sch)
- added sheet rev (rev.kicad_sch)
- note removed: "+"
- note removed: "-"
- note removed: "0x55"
- note removed: "3V REGULATOR"
- note removed: "Battery + header"
- note removed: "Battery connection"
- note removed: "Button0 Right"
- note removed: "Button1 Left"
- note removed: "Button2 Up"
- note removed: "Button3 Down"
- note removed: "Power path output"
- note removed: "System vout"
- note removed: "USB charge in"
- note removed: "USB input"
- note removed: "V_{f} < 3.0V"
- note removed: "charging Power input"
- moved on the sheet: TP1

Commit message: update kicad 9
Parts:
- J1, SW1, SW2, SW3: ID (none) -> 0
- R1, R2: ID 110 -> 10
- TP1: ID (none) -> 0; now not fitted
