File: Hardware/Wireless/dbg.kicad_sch (KiCad schematic)
At the start: 37 parts, among them J6 Conn_01x04_Pin, J7 USB_C_Receptacle_USB2.0, J8 USB_C_Receptacle_USB2.0, U22 STM32F103CBTx, U23 AP2112K-3.3, U24 Conn_01x14_Socket, Y1 32.768KHZ, Y2 8Mhz

Commit message: update kicad 9
Parts:
- C70, C71, C73, C74, C76: value 100nF -> 100nf
- D34, D35: ID 97 -> 126
- J6, JP7, JP8, JP9, U22, U24: ID (none) -> 0
- JP6: ID (none) -> 0; now not fitted
- R47, R48, R49: value 10k -> 10K
Changed lines of the file:
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@@
 (kicad_sch
-	(version 20231120)
+	(version 20250114)
 	(generator "eeschema")
-	(generator_version "8.0")
+	(generator_version "9.0")
 	(paper "A4")
+	(text "Battery + header"
+		(exclude_from_sim no)
+		(at 222.885 158.115 0)
+		(effects
+			(font
+				(size 1.27 1.27)
+			)
+		)
+	)
 	(junction
 		(at 161.29 61.595)
@@
 		)
 	)
-	(text "Battery + header"
-		(exclude_from_sim no)
-		(at 222.885 158.115 0)
-		(effects
-			(font
-				(size 1.27 1.27)
-			)
-		)
-	)
 	(label "PC13"
 		(at 56.515 58.42 180)
-		(fields_autoplaced yes)
 		(effects
 			(font
@@
 	(label "PC13"
 		(at 143.51 121.92 0)
-		(fields_autoplaced yes)
 		(effects
 			(font
@@
 	(label "USBDP"
 		(at 163.195 66.675 0)
-		(fields_autoplaced yes)
 		(effects
 			(font
@@
 	(label "swd"
 		(at 214.63 106.68 180)
-		(fields_autoplaced yes)
 		(effects
 			(font
@@
 	(label "USBDM2"
 		(at 208.28 138.43 0)
-		(fields_autoplaced yes)
 		(effects
 			(font
@@
 	(label "USBDM2"
 		(at 219.075 60.325 0)
-		(fields_autoplaced yes)
 		(effects
 			(font
@@
 	(label "BOOT0"
 		(at 47.625 45.72 180)
-		(fields_autoplaced yes)
 		(effects
 			(font
@@
 	(label "TX"
 		(at 90.17 63.5 0)
-		(fields_autoplaced yes)
 		(effects
 			(font
@@
 	(label "BOOT0"
 		(at 149.86 167.64 270)
-		(fields_autoplaced yes)
 		(effects
 			(font
@@
 	(label "swd"
 		(at 208.28 140.97 0)
-		(fields_autoplaced yes)
 		(effects
 			(font
@@
 	(label "OSCOUT"
 		(at 53.975 50.8 180)
-		(fields_autoplaced yes)
 		(effects
 			(font
@@
 	(label "swd"
 		(at 57.15 104.14 180)
-		(fields_autoplaced yes)
 		(effects
 			(font
@@
 	(label "USBDP2"
 		(at 214.63 99.06 180)
-		(fields_autoplaced yes)
 		(effects
 			(font
@@
 	(label "RX"
 		(at 90.17 66.04 0)
-		(fields_autoplaced yes)
 		(effects
 			(font
@@
 	(label "swc"
 		(at 91.44 53.34 0)
-		(fields_autoplaced yes)
 		(effects
 			(font
@@
 	(label "USBDP2"
 		(at 208.28 133.35 0)
-		(fields_autoplaced yes)
 		(effects
 			(font
@@
 	(label "USBDM"
 		(at 163.195 61.595 0)
-		(fields_autoplaced yes)
 		(effects
 			(font
@@
 	(label "USBDM2"
 		(at 214.63 101.6 180)
-		(fields_autoplaced yes)
 		(effects
 			(font
@@
 	(label "OSCIN"
 		(at 153.035 19.685 0)
-		(fields_autoplaced yes)
 		(effects
 			(font
@@
 	(label "USBDP"
 		(at 118.745 71.12 0)
-		(fields_autoplaced yes)
 		(effects
 			(font
@@
 	(label "BOOT1"
 		(at 48.26 73.66 180)
-		(fields_autoplaced yes)
 		(effects
 			(font
@@
 	(label "OSCOUT"
 		(at 153.035 32.385 0)
-		(fields_autoplaced yes)
 		(effects
 			(font
@@
 	(label "USBDP2"
 		(at 219.075 65.405 0)
-		(fields_autoplaced yes)
 		(effects
 			(font
@@
 	(label "RX"
 		(at 31.75 135.89 180)
-		(fields_autoplaced yes)
 		(effects
 			(font
@@
 	(label "swc"
 		(at 214.63 104.14 180)
-		(fields_autoplaced yes)
 		(effects
 			(font
@@
 	(label "USBDM"
 		(at 102.235 68.58 0)
-		(fields_autoplaced yes)
 		(effects
 			(font
@@
 	(label "TX"
 		(at 31.75 138.43 180)
-		(fields_autoplaced yes)
 		(effects
 			(font
@@
 	(label "swc"
 		(at 208.28 135.89 0)
-		(fields_autoplaced yes)
 		(effects
 			(font
@@
 	(label "BOOT1"
 		(at 149.225 149.225 270)
-		(fields_autoplaced yes)
 		(effects
 			(font
@@
 	(label "OSCIN"
 		(at 53.975 53.34 180)
-		(fields_autoplaced yes)
 		(effects
 			(font
@@
 		(shape input)
 		(at 214.63 104.14 0)
-		(fields_autoplaced yes)
 		(effects
 			(font
@@
 		(shape input)
 		(at 214.63 101.6 0)
-		(fields_autoplaced yes)
 		(effects
 			(font
@@
 		(shape input)
 		(at 214.63 106.68 0)
-		(fields_autoplaced yes)
 		(effects
 			(font
@@
 		(shape input)
 		(at 214.63 109.22 0)
-		(fields_autoplaced yes)
 		(effects
 			(font
@@
 		(shape input)
 		(at 214.63 99.06 0)
-		(fields_autoplaced yes)
 		(effects
 			(font
@@
 		(shape input)
 		(at 214.63 96.52 0)
-		(fields_autoplaced yes)
 		(effects
 			(font
@@
 			)
 		)
+		(property "ID" "0"
+			(at 247.015 107.315 0)
+			(effects
+				(font
+					(size 1.27 1.27)
+				)
+				(hide yes)
+			)
+		)
 		(pin "1"
 		)
@@
 			)
 		)
-		(property "Value" "100nF"
+		(property "Value" "100nf"
 			(at 61.595 156.21 90)
 			(effects
@@
 			)
 		)
-		(property "Value" "10k"
+		(property "Value" "10K"
 			(at 55.245 37.465 0)
 			(effects
@@
 			)
 		)
+		(property "ID" "0"
+			(at 36.83 138.43 0)
+			(effects
+				(font
+					(size 1.27 1.27)
+				)
+				(hide yes)
+			)
+		)
 		(pin "3"
 		)
@@
 			)
 		)
-		(property "Value" "100nF"
+		(property "Value" "100nf"
 			(at 107.95 156.21 90)
 			(effects
@@
 			)
 		)
-		(property "Value" "100nF"
+		(property "Value" "100nf"
 			(at 95.25 27.305 90)
 			(effects
@@
 			)
 		)
-		(property "Value" "10k"
+		(property "Value" "10K"
 			(at 52.07 45.72 90)
 			(effects
@@
 			)
 		)
-		(property "ID" "97"
+		(property "ID" "126"
 			(at 130.81 121.92 0)
 			(effects
@@
 			)
 		)
+		(property "ID" "0"
+			(at 149.225 145.415 0)
+			(effects
+				(font
+					(size 1.27 1.27)
+				)
+				(hide yes)
+			)
+		)
 		(pin "1"
 		)
@@
 			)
 		)
-		(property "Value" "10k"
+		(property "Value" "10K"
 			(at 52.07 71.12 90)
 			(effects
@@
 			)
 		)
+		(property "ID" "0"
+			(at 72.39 76.2 0)
+			(effects
+				(font
+					(size 1.27 1.27)
+				)
+				(hide yes)
+			)
+		)
 		(pin "11"
 		)
@@
 			)
 		)
+		(property "ID" "0"
+			(at 203.2 135.89 0)
+			(effects
+				(font
+					(size 1.27 1.27)
+				)
+				(hide yes)
+			)
+		)
 		(pin "13"
 		)
@@
 			)
 		)
+		(property "ID" "0"
+			(at 149.86 163.83 0)
+			(effects
+				(font
+					(size 1.27 1.27)
+				)
+				(hide yes)
+			)
+		)
 		(pin "1"
 		)
@@
 			)
 		)
-		(property "ID" "97"
+		(property "ID" "126"
 			(at 176.53 153.67 0)
 			(effects
@@
 			)
 		)
-		(property "Value" "100nF"
+		(property "Value" "100nf"
 			(at 33.02 44.45 90)
 			(effects
@@
 			)
 		)
-		(property "Value" "100nF"
+		(property "Value" "100nf"
 			(at 95.885 30.48 90)
 			(effects
@@
 		(in_bom yes)
 		(on_board yes)
-		(dnp no)
+		(dnp yes)
 		(property "Reference" "JP6"
 			(at 30.48 34.925 90)
@@
 			(at 43.18 36.195 0)
 			(effects
+				(font
+					(size 1.27 1.27)
+				)
+				(hide yes)
+			)
+		)
+		(property "ID" "0"
+			(at 43.18 36.195 0)
+			(effects
