File: Hardware/Wireless/pod.kicad_sch (KiCad schematic)
At the start: 145 parts, among them J5 Conn_01x02_Pin, Q10 PMOS-BSS84, Q7 PMOS-BSS84, Q8 IRLML6344, Q9 PMOS-BSS84, SW6 SW_DPDT_x2, U10 battery_charger, U11 nRF52840_aQFN73, U12 TS5A3159AYZPR, U13 BQ27427, U14 TPS22910A, U15 A3144e, U16 A3144e, U18 pogopins, U19 LSM6DS3, U20 TPS54202DDC, U21 TPS54202DDC, X3 32.768 kHz, X4 32MHZ

Commit message: routed
Parts:
- added J9: Conn_01x04_Socket, Connector_PinSocket_2.54mm:PinSocket_1x04_P2.54mm_Vertical, symbol Connector:Conn_01x04_Socket
Connections:
- net 3V: now also J9.2 (Pin_2)
- net GND: now also J9.1 (Pin_1)
- net SCL: now also J9.3 (Pin_3)
- net SDA: now also J9.4 (Pin_4)
Changed lines of the file:
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@@
 		)
 	)
+	(label "SCL"
+		(at -7.62 236.22 270)
+		(fields_autoplaced yes)
+		(effects
+			(font
+				(size 1.27 1.27)
+			)
+			(justify right)
+		)
+		(property "Intersheetrefs" "${INTERSHEET_REFS}"
+			(at -7.62 242.7128 90)
+			(effects
+				(font
+					(size 1.27 1.27)
+				)
+				(justify right)
+				(hide yes)
+			)
+		)
+	)
 	(label "int1"
 		(at 221.615 -20.32 0)
@@
 		)
 	)
+	(label "3V"
+		(at -10.16 236.22 270)
+		(fields_autoplaced yes)
+		(effects
+			(font
+				(size 1.27 1.27)
+			)
+			(justify right)
+		)
+		(property "Intersheetrefs" "${INTERSHEET_REFS}"
+			(at -10.16 239.4391 90)
+			(effects
+				(font
+					(size 1.27 1.27)
+				)
+				(justify right)
+				(hide yes)
+			)
+		)
+	)
 	(label "P0.30"
 		(at 10.795 -6.985 90)
@@
 		)
 	)
+	(label "SDA"
+		(at -5.08 236.22 270)
+		(fields_autoplaced yes)
+		(effects
+			(font
+				(size 1.27 1.27)
+			)
+			(justify right)
+		)
+		(property "Intersheetrefs" "${INTERSHEET_REFS}"
+			(at -5.08 242.7733 90)
+			(effects
+				(font
+					(size 1.27 1.27)
+				)
+				(justify right)
+				(hide yes)
+			)
+		)
+	)
 	(label "MOS_LED_5V"
 		(at 28.575 -6.985 90)
@@
 	)
 	(symbol
+		(lib_id "Connector:Conn_01x04_Socket")
+		(at -10.16 231.14 90)
+		(unit 1)
+		(exclude_from_sim no)
+		(in_bom yes)
+		(on_board yes)
+		(dnp no)
+		(fields_autoplaced yes)
+		(property "Reference" "J9"
+			(at -8.89 226.695 90)
+			(effects
+				(font
+					(size 1.27 1.27)
+				)
+			)
+		)
+		(property "Value" "Conn_01x04_Socket"
+			(at -8.89 229.235 90)
+			(effects
+				(font
+					(size 1.27 1.27)
+				)
+			)
+		)
+		(property "Footprint" "Connector_PinSocket_2.54mm:PinSocket_1x04_P2.54mm_Vertical"
+			(at -10.16 231.14 0)
+			(effects
+				(font
+					(size 1.27 1.27)
+				)
+				(hide yes)
+			)
+		)
+		(property "Datasheet" "~"
+			(at -10.16 231.14 0)
+			(effects
+				(font
+					(size 1.27 1.27)
+				)
+				(hide yes)
+			)
+		)
+		(property "Description" "Generic connector, single row, 01x04, script generated"
+			(at -10.16 231.14 0)
+			(effects
+				(font
+					(size 1.27 1.27)
+				)
+				(hide yes)
+			)
+		)
+		(pin "1"
+		)
+		(pin "3"
+		)
+		(pin "4"
+		)
+		(pin "2"
+		)
+		(instances
+			(project "Revolutetestboard"
+				(path "/e63e39d7-6ac0-4ffd-8aa3-1841a4541b55/23e4cadd-1cee-4e80-b1f8-bbb8e1d83c4a"
+					(reference "J9")
+					(unit 1)
+				)
+			)
+		)
+	)
+	(symbol
 		(lib_id "Library:A3144")
 		(at 138.43 4.445 0)
@@
 					(unit 1)
 				)
+			)
+		)
+	)
+	(symbol
+		(lib_id "nrfmicro-rescue:GND")
+		(at -12.7 236.22 0)
+		(unit 1)
+		(exclude_from_sim no)
+		(in_bom yes)
+		(on_board yes)
+		(dnp no)
+		(property "Reference" "#PWR027"
+			(at -12.7 242.57 0)
+			(effects
+				(font
+					(size 1.27 1.27)
+				)
+				(hide yes)
+			)
+		)
+		(property "Value" "GND"
+			(at -13.97 240.665 0)
+			(effects
+				(font
+					(size 1.27 1.27)
+				)
+			)
+		)
+		(property "Footprint" ""
+			(at -12.7 236.22 0)
+			(effects
+				(font
+					(size 1.27 1.27)
+				)
+				(hide yes)
+			)
+		)
+		(property "Datasheet" ""
+			(at -12.7 236.22 0)
+			(effects
+				(font
+					(size 1.27 1.27)
+				)
+				(hide yes)
+			)
+		)
+		(property "Description" ""
+			(at -12.7 236.22 0)
+			(effects
+				(font
+					(size 1.27 1.27)
+				)
+				(hide yes)
+			)
+		)
+		(pin "1"
+		)
+		(instances
+			(project "Revolutetestboard"
+				(path "/e63e39d7-6ac0-4ffd-8aa3-1841a4541b55/23e4cadd-1cee-4e80-b1f8-bbb8e1d83c4a"
+					(reference "#PWR027")
+					(unit 1)
+				)

Commit message: test board done
Parts:
- removed D3: RED_LED, LED_SMD:LED_0402_1005Metric, symbol Device:LED
- removed R29: 1K, Resistor_SMD:R_0402_1005Metric, symbol Device:R
- added R58, R59, R7: 220r, Resistor_SMD:R_0402_1005Metric, symbol Device:R
- added U26: 1615 RGB SMD LED, Library:1615 RGB SMD LED, symbol Library:1615_RGB_SMD_LED
Connections:
- net 3V: now also U26.3 (+)
- net G-: now reaches U11.B15 (P1.14)
- net G-: now also R58.2
- net R-: now reaches U11.B19 (P1.11)
- net R-: now also R7.1
- net P0.03 renamed B-
- net B-: now also R59.2
- new net: R59.1, U26.4 (B-)
- new net: R7.2, U26.1 (R-)
- new net: R58.1, U26.2 (G-)

Commit message: finished routing
Parts:
- R32: value 50r -> *50r
Connections:
- net RX_TS5A3159AYZPR: now also R32.2, U12.C2; no longer U12.A1
- net com: now also U12.A1; no longer R32.2, U12.C2
Changed lines of the file:
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@@
 	(text "RX OF NRF"
 		(exclude_from_sim no)
-		(at 109.22 214.63 0)
+		(at 69.85 215.9 0)
 		(effects
 			(font
@@
 	(text "POGOPIN+"
 		(exclude_from_sim no)
-		(at 75.565 211.455 0)
+		(at 103.759 214.503 0)
 		(effects
 			(font
@@
 	)
 	(label "COM"
-		(at 79.375 213.995 180)
+		(at 99.695 216.535 0)
 		(fields_autoplaced yes)
 		(effects
@@
 				(size 1.27 1.27)
 			)
-			(justify right)
+			(justify left)
 		)
 		(property "Intersheetrefs" "${INTERSHEET_REFS}"
-			(at 72.3379 213.995 0)
+			(at 104.6679 216.535 0)
 			(effects
 				(font
 					(size 1.27 1.27)
 				)
-				(justify right)
+				(justify left)
 				(hide yes)
 			)
@@
 	)
 	(label "RX_TS5A3159AYZPR"
-		(at 99.695 216.535 0)
+		(at 79.375 213.995 180)
 		(fields_autoplaced yes)
 		(effects
@@
 				(size 1.27 1.27)
 			)
-			(justify left)
+			(justify right)
 		)
 		(property "Intersheetrefs" "${INTERSHEET_REFS}"
-			(at 121.3672 216.535 0)
+			(at 59.767 213.995 0)
 			(effects
 				(font
 					(size 1.27 1.27)
 				)
-				(justify left)
+				(justify right)
 				(hide yes)
 			)
@@
 			)
 		)
-		(property "Value" "50r"
+		(property "Value" "*50r"
 			(at 84.582 218.44 90)
 			(effects

Commit message: update kicad 9
Parts:
- AE2, BT2, BT3, C58, C64, C65, C66, C67, D10, D11, D12, D13, D14, D15, D16, D17, D18, D19, D20, D21, D22, D23, D24, D25, D26, D27, D28, D29, D30, D31, D32, D6, D7, D8, D9, F1, J5, J9, L10, L5, L8, L9, Q10, Q7, Q8, Q9, R18, R19, R21, R22, R23, R24, R27, R32, R39, R40, R42, R44, R58, R59, R7, SW6, U10, U11, U12, U13, U14, U15, U16, U18, U19, U20, U21, U26: ID (none) -> 0
- C32, C35, C38, C39, C46, C47, C48, C54, C62, C63: value 100nF -> 100nf
- C36, C37: ID (none) -> 4
- C57: ID (none) -> 5
- C59: ID 30 -> 21
- C61: ID (none) -> 15
- D2: ID (none) -> 128
- D4: ID (none) -> 126
- D5: ID (none) -> 34
- JP2, JP3, JP4, JP5, TP10, TP11, TP5, TP6, TP7, TP8, TP9, U17: ID (none) -> 0; now not fitted
- L6: ID (none) -> 11
- L7: ID (none) -> 57
- R15, R20, R30: ID (none) -> 19
- R16, R28: ID (none) -> 23
- R17, R25: ID (none) -> 29
- R26: ID (none) -> 54
- R31: value 10k -> 10K; ID 110 -> 7
- R33, R46: ID (none) -> 10
- R34, R38, R45: ID (none) -> 8
- R35, R37: ID (none) -> 7
- R36, R41, R43: ID (none) -> 6
- X3: ID (none) -> 43
- X4: ID (none) -> 33
