File: Hardware/Wired/MainPCB/Revolute.kicad_sch (KiCad schematic)
At the start: 32 parts, among them J1 USB_A, U1 nRF52840_aQFN73, U3 AP2112K-3.3, U4 debug_ports, X1 32MHZ, X2 32.768 kHz

Commit message: current version
Parts:
- removed AE1: Antenna, RF_Antenna:Johanson_2450AT43F0100, symbol Device:Antenna
- removed C14: 1uF, Capacitor_SMD:C_0402_1005Metric, symbol Device:C_Small
- removed C18: 12pF, Capacitor_SMD:C_0402_1005Metric, symbol Device:C_Small
- removed C20, C21: 4.7uF, Capacitor_SMD:C_0402_1005Metric, symbol Device:C_Small
- removed L3: 15nH, Inductor_SMD:L_0402_1005Metric, symbol Device:L
- removed U1: nRF52840_aQFN73, Library:AQFN-73-1EP_7x7mm_P0.5mm_NRF52840-custom, symbol MCU_Nordic:nRF52840_aQFN73
- removed U3: AP2112K-3.3, Package_TO_SOT_SMD:SOT-23-5, symbol Regulator_Linear:AP2112K-3.3
- removed U4: debug_ports, Library:Debug pin cluster, symbol Library:debug_ports
- removed X1: 32MHZ, Library:crystal 32mhz, symbol Device:Crystal_GND24_Small
- removed X2: 32.768 kHz, Crystal:Crystal_SMD_2012-2Pin_2.0x1.2mm, symbol Device:Crystal_Small
- added U1: nrf52833_qfn40, Library:QFN-40-1EP_5x5mm_P0.4mm_EP3.6x3.6mm, symbol Library:nrf52833_qfn40
- added U2: MIC5504, Library:TDFN-4, symbol ESP32-eagle-import:MIC5504
- added X1: 32.768 kHz, Library:Crystal_SMD_2012-2Pin_2.0x1.2mm, symbol Device:Crystal_Small
- added X2: 32MHZ, Library:Crystal_SMD_2016-4Pin_2.0x1.6mm, symbol Device:Crystal_GND24_Small
- C1: value 12pF -> 4.7uF; footprint Capacitor_SMD:C_0402_1005Metric -> Library:Capacitor-0201; ID (none) -> 16
- C10: footprint Capacitor_SMD:C_0402_1005Metric -> Library:Capacitor-0201; ID (none) -> 55
- C11: value 100pF -> 100nF; footprint Capacitor_SMD:C_0402_1005Metric -> Library:Capacitor-0201; ID (none) -> 21
- C12: value 100nF -> 820pF; footprint Capacitor_SMD:C_0402_1005Metric -> Library:Capacitor-0201; ID (none) -> 26
- C13: footprint Capacitor_SMD:C_0402_1005Metric -> Library:Capacitor-0201; ID (none) -> 30
- C15, C16: value 1uF -> 12pF; footprint Capacitor_SMD:C_0402_1005Metric -> Library:Capacitor-0201; ID (none) -> 17
- C17: value 12pF -> 100pF; footprint Capacitor_SMD:C_0402_1005Metric -> Library:Capacitor-0201; ID (none) -> 56
- C2: footprint Capacitor_SMD:C_0402_1005Metric -> Library:Capacitor-0201; ID (none) -> 17
- C3: value 0.8pF -> 12pF; footprint Capacitor_SMD:C_0402_1005Metric -> Library:Capacitor-0201; ID (none) -> 17
- C4: value 0.5pF -> 100nF; footprint Capacitor_SMD:C_0402_1005Metric -> Library:Capacitor-0201; ID (none) -> 21
- C5, C7: value 100nF -> 4.7uF; footprint Capacitor_SMD:C_0402_1005Metric -> Library:Capacitor-0201; ID (none) -> 16
- C6: value 4.7uF -> 1uF; footprint Capacitor_SMD:C_0402_1005Metric -> Library:Capacitor-0201; ID (none) -> 30
- C8: value 100nF -> 1uF; footprint Capacitor_SMD:C_0402_1005Metric -> Library:Capacitor-0201; ID (none) -> 30
- C9: value 820pF -> 1uF; footprint Capacitor_SMD:C_0402_1005Metric -> Library:Capacitor-0201; ID (none) -> 30
- D1: footprint Library:LED_0603_1608Metric-nosilk -> LED_SMD:LED_0402_1005Metric; ID (none) -> 90; JLC Part C72041 -> (none); LCSC Part C146215 -> (none); Manufacturer Part 19-217/BHC-ZL1M2RY/3T -> (none)
- L1: value 4.7nH -> 10uH; ID (none) -> 57
- L2: value 10uH -> 15nH; ID (none) -> 11
- R1: ID (none) -> 27
Connections:
- net BLUE_LED: now also U1.31 (P0.03/AIN1)
- net GND: now also C11.2, C12.1, C15.1, C16.1, C17.1, C2.2, C3.2, C4.2, C6.2, C8.2, C9.2, U1.25 (VSS), U1.37 (VSS), U1.41 (VSS), U2.2 (GND), U2.5 (GND), X2.2, X2.4; no longer C11.1, C12.2, C15.2, C16.2, C17.2, C2.1, C3.1, C4.1, C6.1, C8.1, C9.1
- net VBUS: now also C5.1, C8.1, U1.10 (VBUS), U2.3 (EN), U2.4 (VIN); no longer C13.1
- net VDD_nRF: now also C1.2, C11.1, C13.1, C6.1, U1.18 (VDD), U1.30 (VDD), U1.40 (VDD), U1.8 (VDD), U1.9 (VDDH), U2.1 (VOUT); no longer C12.1, C16.1, C6.2, C7.2, C8.2
- net swc: now also U1.20 (SWDCLK)
- net swd: now also U1.19 (SWDIO)
- net at L1.2: now also U1.39 (DCC); no longer C4.2
- net at L1.1: now also L2.2; no longer C3.2
- net D-: now reaches J1.2 (D-)
- net D-: now also U1.12 (D-)
- net D+: now reaches J1.3 (D+)
- net D+: now also U1.13 (D+)
- net at C10.1: now also C9.1, L2.1, U1.26 (DEC6), U1.38 (DEC4); no longer C15.1
- new net: C7.2, U1.11 (DECUSB)
- new net: C3.1, U1.3 (P0.01/XL2), X1.2
- new net: C4.1, U1.1 (DEC1)
- new net: C2.1, U1.2 (P0.00/XL1), X1.1
- new net: C12.2, U1.21 (DEC5)
- new net: C17.2, U1.27 (DEC3)
- new net: C16.2, U1.28 (XC1), X2.1
- new net: C15.2, U1.29 (XC2), X2.3
- new net ASOUT: U1.7 (P0.11)
- new net DIR: U1.6 (P1.09)
- new net P0.15: U1.14 (P0.15)
- new net P0.17: U1.15 (P0.17)
- new net P0.20: U1.17 (P0.20)
- new net P0.28: U1.33 (P0.28/AIN4)
- new net P0.29: U1.34 (P0.29/AIN5)
- new net P0.30: U1.35 (P0.30/AIN6)
- new net P0.31: U1.36 (P0.31/AIN7)
- new net RESET: U1.16 (P0.18/RESET)
