File: Hardware/RefinedRevolute/Revolute.kicad_pcb (KiCad board)
At the start: 4 copper layers, 19.9 x 19.5 mm, 71 parts, among them J1 -, J2 +, Q1 NMOS-CSD17381F4, Q2 NMOS-CSD17381F4, Q3 PMOS-CSD25483F4, Q4 PMOS-CSD25483F4, Q5 PMOS-CSD25483F4, Q6 PMOS-CSD25483F4, SW1 SW_Omron_B3FS, U1 BQ27427, U2 nrf52833_qfn40, U3 Conn_01x14_Socket, U4 TLV493D, U5 BQ25180, U6 TPS709, U7 TPS22910A, U8 Conn_01x14_Socket, X1 32.768 kHz, X2 32MHZ

Commit message: test board
Parts:
- removed C20: 2.2uF, Capacitor_SMD:C_0603_1608Metric
- added TP3: TestPoint, TestPoint:TestPoint_Pad_D1.0mm, F.Cu at (1.02, 1.02)
- C6: footprint Library:0402 -> Capacitor_SMD:C_0402_1005Metric
- D1: footprint Library:0402 -> LED_SMD:LED_0402_1005Metric
- L1: value 10uH -> Shikues SKSHC0402-100M
- Q1, Q2: value NMOS-CSD17381F4 -> TI CSD17381F4
- Q3, Q4, Q5, Q6: value PMOS-CSD25483F4 -> TI CSD25483F4
- R1, R11, R12, R14, R15, R2, R3, R4, R5, R6, R7, R9, TH1: footprint Library:0402 -> Resistor_SMD:R_0402_1005Metric
- R10, R13, R8: value 10k -> 10K; footprint Library:0402 -> Resistor_SMD:R_0402_1005Metric
- U1: value BQ27427 -> TI BQ27427YZFR
- U2: value nrf52833_qfn40 -> NORDIC nRF52833-QDAA-R
- U3, U8: value Conn_01x14_Socket -> JUSHUO AFH26-S13FIA-1H
- U4: value TLV493D -> Infineon TLV493DA1B6HTSA2
- U5: value BQ25180 -> TI BQ25180YBGR
- U6: value TPS709 -> TI TPS70933DRVT
- U7: value TPS22910A -> TI TPS22910AYZVT
- X1: value 32.768 kHz -> Seiko SC-20S,32.768kHz,20PPM,12.5pF
- X2: value 32MHZ -> NX1612SA-32MHZ-STD-CIS-3
- moved C11 9.95 mm to (154.6, 103.3), turned to 180 degrees
- moved R6 4.24 mm to (147.5, 99.1)
- moved L2 2.96 mm to (148.3, 103.8), turned to -90 degrees
- moved C9 2.82 mm to (147.7, 102.4), turned to 0 degrees
- moved C10 2.66 mm to (147.5, 101.0)
- moved C7 2.27 mm to (149.3, 103.8), turned to 90 degrees
- moved L1 2.06 mm to (147.2, 103.8), turned to 90 degrees
- moved D1 1.13 mm to (147.0, 97.2)
- moved R5 1.06 mm to (148.1, 97.2), turned to -90 degrees
- moved C17 0.93 mm to (143.1, 94.0), turned to 180 degrees
- moved Q6 0.83 mm to (155.4, 104.5)
- moved R7 0.66 mm to (156.5, 104.5)
- moved R8 0.63 mm to (155.2, 105.8)
- moved C15 0.59 mm to (143.5, 95.4)
- moved L3 0.57 mm to (142.5, 95.4), turned to 90 degrees
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Routing:
- net FLEX_LED: track 6.29 -> 1.41 mm, vias 2 -> 0
- net GPOUT: track 12.2 -> 16.7 mm
- net Net-(U3-Pin_1): track 3.05 -> 6.92 mm, vias 0 -> 2
- net tx: track 17.0 -> 19.4 mm
- net Net-(U2-DCC): track 0.88 -> 2.41 mm
- net LOAD_EN: track 16.8 -> 15.6 mm
- net t1: track 8.49 -> 9.63 mm
- net BLUE_LED: track 2.17 -> 1.18 mm
- net Net-(U2-DEC4): track 8.95 -> 9.79 mm
- net Net-(D1-K): track 0.80 -> 1.45 mm
- net GND: track 8.14 -> 7.92 mm, vias 17 -> 13
