File: Hardware/RefinedRevolute/Revolute.kicad_sch (KiCad schematic)
At the start: 72 parts, among them J1 -, J2 +, Q1 NMOS-CSD17381F4, Q2 NMOS-CSD17381F4, Q3 PMOS-CSD25483F4, Q4 PMOS-CSD25483F4, Q5 PMOS-CSD25483F4, Q6 PMOS-CSD25483F4, SW1 SW_Omron_B3FS, U1 BQ27427, U2 nrf52833_qfn40, U3 Conn_01x14_Socket, U4 TLV493D, U5 BQ25180, U6 TPS709, U7 TPS22910A, U8 Conn_01x14_Socket, X1 32.768 kHz, X2 32MHZ

Commit message: test board
Parts:
- C6: footprint Library:0402 -> Capacitor_SMD:C_0402_1005Metric
- D1: footprint Library:0402 -> LED_SMD:LED_0402_1005Metric
- L1: value 10uH -> Shikues SKSHC0402-100M; LCSC (none) -> C18212629
- Q1, Q2: value NMOS-CSD17381F4 -> TI CSD17381F4
- Q3, Q4, Q5, Q6: value PMOS-CSD25483F4 -> TI CSD25483F4
- R1, R10, R11, R12, R13, R14, R15, R2, R3, R4, R5, R6, R7, R8, R9: footprint Library:0402 -> Resistor_SMD:R_0402_1005Metric
- TH1: footprint Library:0402 -> Resistor_SMD:R_0402_1005Metric; LCSC (none) -> C77131
- U1: value BQ27427 -> TI BQ27427YZFR
- U2: value nrf52833_qfn40 -> NORDIC nRF52833-QDAA-R
- U3, U8: value Conn_01x14_Socket -> JUSHUO AFH26-S13FIA-1H
- U4: value TLV493D -> Infineon TLV493DA1B6HTSA2
- U5: value BQ25180 -> TI BQ25180YBGR
- U6: value TPS709 -> TI TPS70933DRVT
- U7: value TPS22910A -> TI TPS22910AYZVT
- X1: value 32.768 kHz -> Seiko SC-20S,32.768kHz,20PPM,12.5pF; LCSC (none) -> C97607
- X2: value 32MHZ -> NX1612SA-32MHZ-STD-CIS-3
Changed lines of the file:
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@@
 			)
 		)
-		(property "Value" "BQ27427"
+		(property "Value" "TI BQ27427YZFR"
 			(at 39.4286 115.57 0)
 			(effects
@@
 			)
 		)
-		(property "Footprint" "Library:0402"
+		(property "Footprint" "Resistor_SMD:R_0402_1005Metric"
 			(at 247.65 55.88 0)
 			(effects
@@
 			)
 		)
+		(property "LCSC" "C77131"
+			(at 247.65 57.15 0)
+			(effects
+				(font
+					(size 1.27 1.27)
+				)
+				(hide yes)
+			)
+		)
 		(pin "1"
 		)
@@
 			)
 		)
-		(property "Footprint" "Library:0402"
+		(property "Footprint" "Resistor_SMD:R_0402_1005Metric"
 			(at 186.69 122.555 0)
 			(effects
@@
 			)
 		)
-		(property "Value" "PMOS-CSD25483F4"
+		(property "Value" "TI CSD25483F4"
 			(at 87.249 157.988 0)
 			(effects
@@
 			)
 		)
-		(property "Footprint" "Library:0402"
+		(property "Footprint" "Capacitor_SMD:C_0402_1005Metric"
 			(at 59.055 126.365 0)
 			(effects
@@
 			)
 		)
-		(property "Footprint" "Library:0402"
+		(property "Footprint" "Resistor_SMD:R_0402_1005Metric"
 			(at 187.833 85.09 90)
 			(effects
@@
 			)
 		)
-		(property "Value" "Conn_01x14_Socket"
+		(property "Value" "JUSHUO AFH26-S13FIA-1H"
 			(at 174.244 159.512 0)
 			(effects
@@
 			)
 		)
-		(property "Footprint" "Library:0402"
+		(property "Footprint" "Resistor_SMD:R_0402_1005Metric"
 			(at 187.325 140.335 0)
 			(effects
@@
 			)
 		)
-		(property "Footprint" "Library:0402"
+		(property "Footprint" "Resistor_SMD:R_0402_1005Metric"
 			(at 203.2 39.37 0)
 			(effects
@@
 			)
 		)
-		(property "Value" "32.768 kHz"
+		(property "Value" "Seiko SC-20S,32.768kHz,20PPM,12.5pF"
 			(at 35.814 60.452 90)
 			(effects
@@
 			)
 		)
+		(property "LCSC" "C97607"
+			(at 56.515 64.135 90)
+			(effects
+				(font
+					(size 1.27 1.27)
+				)
+				(hide yes)
+			)
+		)
 		(pin "1"
 		)
@@
 			)
 		)
-		(property "Value" "TPS709"
+		(property "Value" "TI TPS70933DRVT"
 			(at 229.235 118.11 0)
 			(effects
@@
 			)
 		)
-		(property "Footprint" "Library:0402"
+		(property "Footprint" "Resistor_SMD:R_0402_1005Metric"
 			(at 137.795 104.14 0)
 			(effects
@@
 			)
 		)
-		(property "Footprint" "Library:0402"
+		(property "Footprint" "Resistor_SMD:R_0402_1005Metric"
 			(at 127 136.525 0)
 			(effects
@@
 			)
 		)
-		(property "Footprint" "Library:0402"
+		(property "Footprint" "Resistor_SMD:R_0402_1005Metric"
 			(at 78.105 152.4 0)
 			(effects
@@
 			)
 		)
-		(property "Footprint" "Library:0402"
+		(property "Footprint" "Resistor_SMD:R_0402_1005Metric"
 			(at 199.39 49.53 0)
 			(effects
@@
 			)
 		)
-		(property "Footprint" "Library:0402"
+		(property "Footprint" "Resistor_SMD:R_0402_1005Metric"
 			(at 139.065 133.35 0)
 			(effects
@@
 			)
 		)
-		(property "Value" "NMOS-CSD17381F4"
+		(property "Value" "TI CSD17381F4"
 			(at 61.595 154.432 0)
 			(effects
@@
 			)
 		)
-		(property "Footprint" "Library:0402"
+		(property "Footprint" "Resistor_SMD:R_0402_1005Metric"
 			(at 151.765 156.845 0)
 			(effects
@@
 			)
 		)
-		(property "Footprint" "Library:0402"
+		(property "Footprint" "Resistor_SMD:R_0402_1005Metric"
 			(at 26.67 122.555 0)
 			(effects
@@
 			)
 		)
-		(property "Value" "BQ25180"
+		(property "Value" "TI BQ25180YBGR"
 			(at 223.52 20.32 0)
 			(effects
@@
 		(exclude_from_sim no)
 		(in_bom yes)
-		(on_board yes)
+		(on_board no)
 		(dnp yes)
 		(property "Reference" "C20"
@@
 			)
 		)
-		(property "Value" "PMOS-CSD25483F4"
+		(property "Value" "TI CSD25483F4"
 			(at 180.975 111.76 0)
 			(effects
@@
 			)
 		)
-		(property "Value" "PMOS-CSD25483F4"
+		(property "Value" "TI CSD25483F4"
 			(at 146.05 133.604 90)
 			(effects
@@
 			)
 		)
-		(property "Value" "nrf52833_qfn40"
+		(property "Value" "NORDIC nRF52833-QDAA-R"
 			(at 90.17 71.755 0)
 			(effects
@@
 			)
 		)
-		(property "Value" "NMOS-CSD17381F4"
+		(property "Value" "TI CSD17381F4"
 			(at 65.405 177.038 0)
 			(effects
@@
 			)
 		)
-		(property "Value" "10uH"
+		(property "Value" "Shikues SKSHC0402-100M"
 			(at 78.74 27.3049 0)
 			(effects
@@
 			)
 		)
+		(property "LCSC" "C18212629"
+			(at 77.47 26.035 0)
+			(effects
+				(font
+					(size 1.27 1.27)
+				)
+				(hide yes)
+			)
+		)
 		(pin "1"
 		)
@@
 			)
 		)
-		(property "Value" "32MHZ"
+		(property "Value" "NX1612SA-32MHZ-STD-CIS-3"
 			(at 128.27 43.18 90)
 			(effects
@@
 			)
 		)
-		(property "Footprint" "Library:0402"
+		(property "Footprint" "Resistor_SMD:R_0402_1005Metric"
 			(at 193.04 40.64 0)
 			(effects
@@
 			)
 		)
-		(property "Value" "TLV493D"
+		(property "Value" "Infineon TLV493DA1B6HTSA2"
 			(at 209.042 84.963 0)
 			(effects
@@
 			)
 		)
-		(property "Footprint" "Library:0402"
+		(property "Footprint" "LED_SMD:LED_0402_1005Metric"
 			(at 130.175 104.14 90)
 			(effects
@@
 			)
 		)
-		(property "Value" "PMOS-CSD25483F4"
+		(property "Value" "TI CSD25483F4"
 			(at 85.979 179.578 0)
 			(effects
@@
 			)
 		)
-		(property "Value" "Conn_01x14_Socket"
+		(property "Value" "JUSHUO AFH26-S13FIA-1H"
 			(at 131.699 166.497 0)
 			(effects
@@
 			)
 		)
-		(property "Footprint" "Library:0402"
+		(property "Footprint" "Resistor_SMD:R_0402_1005Metric"
 			(at 187.833 95.25 90)
 			(effects
@@
 			)
 		)
-		(property "Footprint" "Library:0402"
+		(property "Footprint" "Resistor_SMD:R_0402_1005Metric"
 			(at 78.105 186.69 0)
 			(effects
@@
 			)
 		)
-		(property "Footprint" "Library:0402"
+		(property "Footprint" "Resistor_SMD:R_0402_1005Metric"
 			(at 171.45 116.205 0)
 			(effects
@@
 			)
 		)
-		(property "Value" "TPS22910A"
+		(property "Value" "TI TPS22910AYZVT"
 			(at 233.68 144.526 0)
 			(effects
